File: KiCad/AppAudio.sch (KiCad schematic (older format))
At the start: 1 part, among them U1 TWE_LITE_SMD

Commit message: Writing a schematic diagram.
Parts:
- added C1: 33u, symbol CP
- added C2: 0.1u, symbol C_Small
- added C3: 220u, symbol CP
- added C4: 3300p, symbol C_Small
- added C5: 1000p, symbol C_Small
- added C6: C, symbol C
- added R1, R2, R6: 10k, symbol R
- added R3: 1.5k, symbol R
- added R4: 1k, symbol R
- added R5: 57k, symbol R
- added R7, R8, R9: 22k, symbol R
- added SW1: SPST, symbol SPST
- added SW2: SW_PUSH, symbol SW_PUSH
- added U2: MIC_ELECTRET, symbol MIC_ELECTRET
- added U3: LMC6062, symbol LMC6062
- added VR1: 50k, symbol POT
- added VR2: 1k, symbol POT
Connections:
- net labels added: GND, VCC
- wire segments 0 -> 59

Commit message: PCB layout in progress.
Parts:
- removed SW1: SPST, symbol SPST
- added BT1: Battery, symbol Battery
- added C7: 1u, Capacitors_ThroughHole:C_Rect_L4_W2.5_P2.5, symbol C
- added D1: Led_x2, LEDs:LED-5MM-3, symbol Led_x2
- added P1: WRITER-VCC, favorites:WRITE-7P, symbol WRITER-VCC
- added Q1: Q_NMOS_SGD, favorites:EMT3, symbol Q_NMOS_SGD
- added R10, R13: 1k, Resistors_ThroughHole:Resistor_Horizontal_RM10mm, symbol R
- added R11, R12: 2.2M, Resistors_ThroughHole:Resistor_Horizontal_RM10mm, symbol R
- added SP1: SPEAKER, Pin_Headers:Pin_Header_Straight_1x02, symbol SPEAKER
- added SW1: SWITCH_INV, Terminal_Blocks:TerminalBlock_WAGO-236_2Stift_RM5mm_3pol, symbol SWITCH_INV
- added U3: HT82V739, Housings_DIP:DIP-8_W7.62mm, symbol HT82V739
- C1, C3: footprint (none) -> Capacitors_ThroughHole:C_Radial_D5_L6_P2.5
- C2, C4, C5: footprint (none) -> Capacitors_ThroughHole:C_Rect_L4_W2.5_P2.5
- C6: value C -> 22u; footprint (none) -> Capacitors_ThroughHole:C_Radial_D5_L6_P2.5
- MIC1: renamed from U2; footprint (none) -> Capacitors_ThroughHole:C_Radial_D6.3_L11.2_P2.5
- R1, R2, R3, R4, R5, R6, R7, R8: footprint (none) -> Resistors_ThroughHole:Resistor_Horizontal_RM10mm
- R9: value 22k -> 100; footprint (none) -> Resistors_ThroughHole:Resistor_Horizontal_RM10mm
- SW2: footprint (none) -> favorites:JB-15HFBP2
- U1: footprint MODULE -> favorites:TWE-001L-NC7
- U2: renamed from U3; footprint (none) -> Housings_DIP:DIP-8_W7.62mm
- VR1, VR2: footprint (none) -> favorites:RV-TSR-3386T
Connections:
- net labels added: CFG, PRG, QGND, RST, RXD, TXD, VSS
- wire segments 59 -> 117
- no-connect marks 0 -> 19
Other:
- moved on the sheet: U2B

Commit message: PCB design in progress.
Parts:
- removed SW1: SWITCH_INV, Terminal_Blocks:TerminalBlock_WAGO-236_2Stift_RM5mm_3pol, symbol SWITCH_INV
- added SW2: SW_PUSH, favorites:DTS-6, symbol SW_PUSH
- R10, R13, R4: footprint Resistors_ThroughHole:Resistor_Horizontal_RM10mm -> Resistors_SMD:R_0603_HandSoldering
- VR1, VR2: footprint favorites:RV-TSR-3386T -> favorites:RV-3362P
- renumbered SW2 to SW1
Connections:
- no-connect marks 19 -> 18
Changed lines of the file:
@@
 F 1 "TWE_LITE_SMD" H 5000 3400 50  0000 C CNN
 F 2 "favorites:TWE-001L-NC7" H 4750 1350 50  0001 C CNN
-F 3 "DOCUMENTATION" H 5350 1350 50  0001 C CNN
+F 3 "http://mono-wireless.com/jp/products/TWE-Lite/MNO-PDS-TWE001L-JP-2.10-2.pdf" H 5350 1350 50  0001 C CNN
 	1    5000 2600
 	1    0    0    -1
@@
 F 0 "R4" V 2180 3700 50  0000 C CNN
 F 1 "1k" V 2100 3700 50  0000 C CNN
-F 2 "Resistors_ThroughHole:Resistor_Horizontal_RM10mm" V 2030 3700 50  0001 C CNN
+F 2 "Resistors_SMD:R_0603_HandSoldering" V 2030 3700 50  0001 C CNN
 F 3 "" H 2100 3700 50  0000 C CNN
 	1    2100 3700
@@
 L GND #PWR03
 U 1 1 5716320D
-P 3750 4750
-F 0 "#PWR03" H 3750 4500 50  0001 C CNN
-F 1 "GND" H 3750 4600 50  0000 C CNN
-F 2 "" H 3750 4750 50  0000 C CNN
-F 3 "" H 3750 4750 50  0000 C CNN
-	1    3750 4750
+P 3650 4350
+F 0 "#PWR03" H 3650 4100 50  0001 C CNN
+F 1 "GND" H 3650 4200 50  0000 C CNN
+F 2 "" H 3650 4350 50  0000 C CNN
+F 3 "" H 3650 4350 50  0000 C CNN
+	1    3650 4350
 	1    0    0    -1
 $EndComp
@@
 F 0 "VR1" H 3150 1870 50  0000 C CNN
 F 1 "50k" H 3150 1950 50  0000 C CNN
-F 2 "favorites:RV-TSR-3386T" H 3150 1950 50  0001 C CNN
+F 2 "favorites:RV-3362P" H 3150 1950 50  0001 C CNN
 F 3 "" H 3150 1950 50  0000 C CNN
 	1    3150 1950
@@
 F 0 "VR2" H 6300 3020 50  0000 C CNN
 F 1 "1k" H 6300 3100 50  0000 C CNN
-F 2 "favorites:RV-TSR-3386T" H 6300 3100 50  0001 C CNN
+F 2 "favorites:RV-3362P" H 6300 3100 50  0001 C CNN
 F 3 "" H 6300 3100 50  0000 C CNN
 	1    6300 3100
@@
 $EndComp
 $Comp
-L SW_PUSH SW2
+L SW_PUSH SW1
 U 1 1 5716980D
 P 3350 3700
-F 0 "SW2" H 3500 3810 50  0000 C CNN
+F 0 "SW1" H 3500 3810 50  0000 C CNN
 F 1 "SW_PUSH" H 3350 3620 50  0000 C CNN
 F 2 "favorites:JB-15HFBP2" H 3350 3700 50  0001 C CNN
@@
 F 0 "R10" V 6180 4750 50  0000 C CNN
 F 1 "1k" V 6100 4750 50  0000 C CNN
-F 2 "Resistors_ThroughHole:Resistor_Horizontal_RM10mm" V 6030 4750 50  0001 C CNN
+F 2 "Resistors_SMD:R_0603_HandSoldering" V 6030 4750 50  0001 C CNN
 F 3 "" H 6100 4750 50  0000 C CNN
 	1    6100 4750
@@
 F 0 "R13" V 6680 2600 50  0000 C CNN
 F 1 "1k" V 6600 2600 50  0000 C CNN
-F 2 "Resistors_ThroughHole:Resistor_Horizontal_RM10mm" V 6530 2600 50  0001 C CNN
+F 2 "Resistors_SMD:R_0603_HandSoldering" V 6530 2600 50  0001 C CNN
 F 3 "" H 6600 2600 50  0000 C CNN
 	1    6600 2600
@@
 Text Label 6700 4600 0    60   ~ 0
 QGND
-$Comp
-L SWITCH_INV SW1
-U 1 1 571ABE3F
-P 3650 4150
-F 0 "SW1" H 3450 4300 50  0000 C CNN
-F 1 "SWITCH_INV" H 3500 4000 50  0000 C CNN
-F 2 "Terminal_Blocks:TerminalBlock_WAGO-236_2Stift_RM5mm_3pol" H 3650 4150 50  0001 C CNN
-F 3 "" H 3650 4150 50  0000 C CNN
-	1    3650 4150
-	0    1    1    0
-$EndComp
-Wire Wire Line
-	3750 4750 3750 4650
-NoConn ~ 3550 4650
+Wire Wire Line
+	3650 4350 3650 4250
 $Comp
 L Battery BT1
@@
 	8350 1750 8000 1750
 Connection ~ 8000 1750
+$Comp
+L SW_PUSH SW2
+U 1 1 5725EDAD
+P 3650 3950
+F 0 "SW2" H 3800 4060 50  0000 C CNN
+F 1 "SW_PUSH" H 3650 3870 50  0000 C CNN
+F 2 "favorites:DTS-6" H 3650 3950 50  0001 C CNN
+F 3 "" H 3650 3950 50  0000 C CNN
+	1    3650 3950
+	0    -1   1    0
+$EndComp
 $EndSCHEMATC
