File: KiCad/AppAudio.sch (KiCad schematic (older format))
At the start: 33 parts, among them P1 WRITER-VCC, Q1 Q_NMOS_SGD, SW1 SW_PUSH, SW2 SW_PUSH, U1 TWE_LITE_SMD, U2 LMC6062, U3 HT82V739

Commit message: Fixed wires.
Connections:
- wire segments 115 -> 117

Commit message: PCB layout has done.
Parts:
- BT1: footprint (none) -> Pin_Headers:Pin_Header_Straight_1x02
- C3, C6: footprint Capacitors_ThroughHole:C_Radial_D5_L6_P2.5 -> Capacitors_ThroughHole:C_Radial_D6.3_L11.2_P2.5
- MIC1: footprint Capacitors_ThroughHole:C_Radial_D6.3_L11.2_P2.5 -> favorites:DB-C9767
Changed lines of the file:
@@
 F 0 "MIC1" H 1000 3050 60  0000 C CNN
 F 1 "MIC_ELECTRET" H 1000 2450 60  0000 C CNN
-F 2 "Capacitors_ThroughHole:C_Radial_D6.3_L11.2_P2.5" H 1000 2800 60  0001 C CNN
+F 2 "favorites:DB-C9767" H 1000 2800 60  0001 C CNN
 F 3 "" H 1000 2800 60  0000 C CNN
 	1    1000 2800
@@
 F 0 "C3" H 8025 1450 50  0000 L CNN
 F 1 "220u" H 8025 1250 50  0000 L CNN
-F 2 "Capacitors_ThroughHole:C_Radial_D5_L6_P2.5" H 8038 1200 50  0001 C CNN
+F 2 "Capacitors_ThroughHole:C_Radial_D6.3_L11.2_P2.5" H 8038 1200 50  0001 C CNN
 F 3 "" H 8000 1350 50  0000 C CNN
 	1    8000 1350
@@
 F 0 "C6" H 8725 3300 50  0000 L CNN
 F 1 "22u" H 8725 3100 50  0000 L CNN
-F 2 "Capacitors_ThroughHole:C_Radial_D5_L6_P2.5" H 8738 3050 50  0001 C CNN
+F 2 "Capacitors_ThroughHole:C_Radial_D6.3_L11.2_P2.5" H 8738 3050 50  0001 C CNN
 F 3 "" H 8700 3200 50  0000 C CNN
 	1    8700 3200
@@
 F 0 "BT1" H 7500 1350 50  0000 L CNN
 F 1 "Battery" H 7500 1250 50  0000 L CNN
-F 2 "" V 7400 1340 50  0000 C CNN
+F 2 "Pin_Headers:Pin_Header_Straight_1x02" V 7400 1340 50  0000 C CNN
 F 3 "" V 7400 1340 50  0000 C CNN
 	1    7400 1300

Commit message: Changed the footprint of the LED.
Parts:
- D1: footprint LEDs:LED-5MM-3 -> favorites:LED-3MM
Changed lines of the file:
@@
 F 0 "D1" H 6250 2575 50  0000 C CNN
 F 1 "Led_x2" H 6250 2100 50  0000 C CNN
-F 2 "LEDs:LED-5MM-3" H 6250 2350 50  0001 C CNN
+F 2 "favorites:LED-3MM" H 6250 2350 50  0001 C CNN
 F 3 "" H 6250 2350 50  0000 C CNN
 	1    6250 2350

Commit message: Added the 3d model of the speaker.
Parts:
- BT1, SP1: footprint Pin_Headers:Pin_Header_Straight_1x02 -> favorites:B02B-XASK-1
- R1, R2, R3, R5, R6, R7, R8: footprint Resistors_ThroughHole:Resistor_Horizontal_RM10mm -> Resistors_SMD:R_0603_HandSoldering
- SW1: footprint favorites:JB-15HFBP2 -> favorites:TVGP01-G73BB
- SW2: footprint favorites:DTS-6 -> favorites:JB-15HFBP2
Connections:
- net labels added: Aud_In, OUTN, OUTP, VREF
Changed lines of the file:
@@
 F 0 "R1" V 1530 2400 50  0000 C CNN
 F 1 "10k" V 1450 2400 50  0000 C CNN
-F 2 "Resistors_ThroughHole:Resistor_Horizontal_RM10mm" V 1380 2400 50  0001 C CNN
+F 2 "Resistors_SMD:R_0603_HandSoldering" V 1380 2400 50  0001 C CNN
 F 3 "" H 1450 2400 50  0000 C CNN
 	1    1450 2400
@@
 F 0 "R2" V 2180 2700 50  0000 C CNN
 F 1 "10k" V 2100 2700 50  0000 C CNN
-F 2 "Resistors_ThroughHole:Resistor_Horizontal_RM10mm" V 2030 2700 50  0001 C CNN
+F 2 "Resistors_SMD:R_0603_HandSoldering" V 2030 2700 50  0001 C CNN
 F 3 "" H 2100 2700 50  0000 C CNN
 	1    2100 2700
@@
 F 0 "R3" V 2180 3300 50  0000 C CNN
 F 1 "1.5k" V 2100 3300 50  0000 C CNN
-F 2 "Resistors_ThroughHole:Resistor_Horizontal_RM10mm" V 2030 3300 50  0001 C CNN
+F 2 "Resistors_SMD:R_0603_HandSoldering" V 2030 3300 50  0001 C CNN
 F 3 "" H 2100 3300 50  0000 C CNN
 	1    2100 3300
@@
 F 0 "R5" V 2630 1950 50  0000 C CNN
 F 1 "57k" V 2550 1950 50  0000 C CNN
-F 2 "Resistors_ThroughHole:Resistor_Horizontal_RM10mm" V 2480 1950 50  0001 C CNN
+F 2 "Resistors_SMD:R_0603_HandSoldering" V 2480 1950 50  0001 C CNN
 F 3 "" H 2550 1950 50  0000 C CNN
 	1    2550 1950
@@
 F 0 "R6" V 3580 1950 50  0000 C CNN
 F 1 "10k" V 3500 1950 50  0000 C CNN
-F 2 "Resistors_ThroughHole:Resistor_Horizontal_RM10mm" V 3430 1950 50  0001 C CNN
+F 2 "Resistors_SMD:R_0603_HandSoldering" V 3430 1950 50  0001 C CNN
 F 3 "" H 3500 1950 50  0000 C CNN
 	1    3500 1950
@@
 F 0 "R7" V 6780 3100 50  0000 C CNN
 F 1 "22k" V 6700 3100 50  0000 C CNN
-F 2 "Resistors_ThroughHole:Resistor_Horizontal_RM10mm" V 6630 3100 50  0001 C CNN
+F 2 "Resistors_SMD:R_0603_HandSoldering" V 6630 3100 50  0001 C CNN
 F 3 "" H 6700 3100 50  0000 C CNN
 	1    6700 3100
@@
 F 0 "R8" V 7180 3100 50  0000 C CNN
 F 1 "22k" V 7100 3100 50  0000 C CNN
-F 2 "Resistors_ThroughHole:Resistor_Horizontal_RM10mm" V 7030 3100 50  0001 C CNN
+F 2 "Resistors_SMD:R_0603_HandSoldering" V 7030 3100 50  0001 C CNN
 F 3 "" H 7100 3100 50  0000 C CNN
 	1    7100 3100
@@
 F 0 "SW1" H 3500 3810 50  0000 C CNN
 F 1 "SW_PUSH" H 3350 3620 50  0000 C CNN
-F 2 "favorites:JB-15HFBP2" H 3350 3700 50  0001 C CNN
+F 2 "favorites:TVGP01-G73BB" H 3350 3700 50  0001 C CNN
 F 3 "" H 3350 3700 50  0000 C CNN
 	1    3350 3700
@@
 F 0 "SP1" H 10600 3500 50  0000 C CNN
 F 1 "SPEAKER" H 10600 3000 50  0000 C CNN
-F 2 "Pin_Headers:Pin_Header_Straight_1x02" H 10700 3250 50  0001 C CNN
+F 2 "favorites:B02B-XASK-1" H 10700 3250 50  0001 C CNN
 F 3 "" H 10700 3250 50  0000 C CNN
 	1    10700 3250
-	1    0    0    -1
+	1    0    0    1
 $EndComp
 $Comp
@@
 F 0 "BT1" H 7500 1350 50  0000 L CNN
 F 1 "Battery" H 7500 1250 50  0000 L CNN
-F 2 "Pin_Headers:Pin_Header_Straight_1x02" V 7400 1340 50  0000 C CNN
+F 2 "favorites:B02B-XASK-1" V 7400 1340 50  0000 C CNN
 F 3 "" V 7400 1340 50  0000 C CNN
 	1    7400 1300
@@
 F 0 "SW2" H 3800 4060 50  0000 C CNN
 F 1 "SW_PUSH" H 3650 3870 50  0000 C CNN
-F 2 "favorites:DTS-6" H 3650 3950 50  0001 C CNN
+F 2 "favorites:JB-15HFBP2" H 3650 3950 50  0001 C CNN
 F 3 "" H 3650 3950 50  0000 C CNN
 	1    3650 3950
@@
 Wire Wire Line
 	3350 4550 3350 4000
+Text Label 10300 3150 0    60   ~ 0
+OUTN
+Text Label 10250 3250 0    60   ~ 0
+OUTP
+Text Label 8850 3200 0    60   ~ 0
+Aud_In
+Text Label 8900 3300 0    60   ~ 0
+VREF
 $EndSCHEMATC

Commit message: Replaced the footprint of SW2.
Parts:
- SW2: footprint favorites:JB-15HFBP2 -> favorites:TVGP01-G73BB
Changed lines of the file:
@@
 F 0 "SW2" H 3800 4060 50  0000 C CNN
 F 1 "SW_PUSH" H 3650 3870 50  0000 C CNN
-F 2 "favorites:JB-15HFBP2" H 3650 3950 50  0001 C CNN
+F 2 "favorites:TVGP01-G73BB" H 3650 3950 50  0001 C CNN
 F 3 "" H 3650 3950 50  0000 C CNN
 	1    3650 3950

Commit message: Removed the net file.
Parts:
- SW2: footprint favorites:TVGP01-G73BB -> favorites:JB-15HFBP2
Changed lines of the file:
@@
 L GND #PWR03
 U 1 1 5716320D
-P 3650 4350
-F 0 "#PWR03" H 3650 4100 50  0001 C CNN
-F 1 "GND" H 3650 4200 50  0000 C CNN
-F 2 "" H 3650 4350 50  0000 C CNN
-F 3 "" H 3650 4350 50  0000 C CNN
-	1    3650 4350
+P 3350 4350
+F 0 "#PWR03" H 3350 4100 50  0001 C CNN
+F 1 "GND" H 3350 4200 50  0000 C CNN
+F 2 "" H 3350 4350 50  0000 C CNN
+F 3 "" H 3350 4350 50  0000 C CNN
+	1    3350 4350
 	1    0    0    -1
 $EndComp
@@
 L GND #PWR04
 U 1 1 5716325B
-P 3350 4550
-F 0 "#PWR04" H 3350 4300 50  0001 C CNN
-F 1 "GND" H 3350 4400 50  0000 C CNN
-F 2 "" H 3350 4550 50  0000 C CNN
-F 3 "" H 3350 4550 50  0000 C CNN
-	1    3350 4550
+P 3050 4550
+F 0 "#PWR04" H 3050 4300 50  0001 C CNN
+F 1 "GND" H 3050 4400 50  0000 C CNN
+F 2 "" H 3050 4550 50  0000 C CNN
+F 3 "" H 3050 4550 50  0000 C CNN
+	1    3050 4550
 	1    0    0    -1
 $EndComp
@@
 L SW_PUSH SW1
 U 1 1 5716980D
-P 3350 3700
-F 0 "SW1" H 3500 3810 50  0000 C CNN
-F 1 "SW_PUSH" H 3350 3620 50  0000 C CNN
-F 2 "favorites:TVGP01-G73BB" H 3350 3700 50  0001 C CNN
-F 3 "" H 3350 3700 50  0000 C CNN
-	1    3350 3700
+P 3050 3700
+F 0 "SW1" H 3200 3810 50  0000 C CNN
+F 1 "SW_PUSH" H 3050 3620 50  0000 C CNN
+F 2 "favorites:TVGP01-G73BB" H 3050 3700 50  0001 C CNN
+F 3 "" H 3050 3700 50  0000 C CNN
+	1    3050 3700
 	0    -1   1    0
 $EndComp
@@
 L SW_PUSH SW2
 U 1 1 5725EDAD
-P 3650 3950
-F 0 "SW2" H 3800 4060 50  0000 C CNN
-F 1 "SW_PUSH" H 3650 3870 50  0000 C CNN
-F 2 "favorites:TVGP01-G73BB" H 3650 3950 50  0001 C CNN
-F 3 "" H 3650 3950 50  0000 C CNN
-	1    3650 3950
+P 3350 3950
+F 0 "SW2" H 3500 4060 50  0000 C CNN
+F 1 "SW_PUSH" H 3350 3870 50  0000 C CNN
+F 2 "favorites:JB-15HFBP2" H 3350 3950 50  0001 C CNN
+F 3 "" H 3350 3950 50  0000 C CNN
+	1    3350 3950
 	0    -1   1    0
 $EndComp
@@
 Connection ~ 8000 1750
 Wire Wire Line
-	8350 1750 8000 1750
+	8000 1750 8350 1750
 Wire Wire Line
 	6300 3350 6450 3350
@@
 	7400 1150 7400 1100
 Wire Wire Line
-	3650 4350 3650 4250
+	3350 4250 3350 4350
 Wire Wire Line
 	6600 2800 6600 2750
@@
 	5750 2450 5950 2450
 Wire Wire Line
-	3650 3350 4250 3350
-Wire Wire Line
-	3650 3650 3650 3350
+	3350 3350 4250 3350
+Wire Wire Line
+	3350 3650 3350 3350
 Connection ~ 9000 3500
 Wire Wire Line
@@
 Connection ~ 8850 4000
 Wire Wire Line
-	9000 3400 9000 4000
-Wire Wire Line
-	9050 3400 9000 3400
-Wire Wire Line
-	9000 4000 8550 4000
+	9000 4000 9000 3400
+Wire Wire Line
+	9000 3400 9050 3400
+Wire Wire Line
+	8550 4000 9000 4000
 Wire Wire Line
 	8850 3950 8850 4000
@@
 	7300 3900 7300 3500
 Wire Wire Line
-	4250 3250 3350 3250
-Wire Wire Line
-	3350 3250 3350 3400
-Wire Wire Line
-	3350 4550 3350 4000
+	4250 3250 3050 3250
+Wire Wire Line
+	3050 3250 3050 3400
+Wire Wire Line
+	3050 4550 3050 4000
 Text Label 10300 3150 0    60   ~ 0
 OUTN

Commit message: Connect CE# to DO3.
Parts:
- C1: value 33u -> 22u; footprint Capacitors_ThroughHole:C_Radial_D5_L6_P2.5 -> Capacitors_ThroughHole:C_Radial_D6.3_L11.2_P2.5; symbol CP -> C_Small
- R11, R12: value 2.2M -> 100k
- U2: value LMC6062 -> NJM13404
Connections:
- net labels added: DO3
- wire segments 117 -> 129
- no-connect marks 18 -> 14
Changed lines of the file:
@@
 $EndComp
 $Comp
-L CP C1
+L C_Small C1
 U 1 1 57162E7C
 P 1700 2700
 F 0 "C1" H 1725 2800 50  0000 L CNN
-F 1 "33u" H 1725 2600 50  0000 L CNN
-F 2 "Capacitors_ThroughHole:C_Radial_D5_L6_P2.5" H 1738 2550 50  0001 C CNN
+F 1 "22u" H 1725 2600 50  0000 L CNN
+F 2 "Capacitors_ThroughHole:C_Radial_D6.3_L11.2_P2.5" H 1738 2550 50  0001 C CNN
 F 3 "" H 1700 2700 50  0000 C CNN
 	1    1700 2700
@@
 P 2700 2800
 F 0 "U2" H 2650 3000 50  0000 L CNN
-F 1 "LMC6062" H 2650 2550 50  0000 L CNN
+F 1 "NJM13404" H 2650 2550 50  0000 L CNN
 F 2 "Housings_DIP:DIP-8_W7.62mm" H 2700 2800 50  0001 C CNN
 F 3 "" H 2700 2800 50  0000 C CNN
@@
 L POT VR2
 U 1 1 571641D3
-P 6300 3100
-F 0 "VR2" H 6300 3020 50  0000 C CNN
-F 1 "1k" H 6300 3100 50  0000 C CNN
-F 2 "favorites:RV-3362P" H 6300 3100 50  0001 C CNN
-F 3 "" H 6300 3100 50  0000 C CNN
-	1    6300 3100
+P 6350 3100
+F 0 "VR2" H 6350 3020 50  0000 C CNN
+F 1 "1k" H 6350 3100 50  0000 C CNN
+F 2 "favorites:RV-3362P" H 6350 3100 50  0001 C CNN
+F 3 "" H 6350 3100 50  0000 C CNN
+	1    6350 3100
 	0    1    1    0
 $EndComp
@@
 P 7750 3200
 F 0 "U2" H 7700 3400 50  0000 L CNN
-F 1 "LMC6062" H 7700 2950 50  0000 L CNN
+F 1 "NJM13404" H 7700 2950 50  0000 L CNN
 F 2 "Housings_DIP:DIP-8_W7.62mm" H 7750 3200 50  0001 C CNN
 F 3 "" H 7750 3200 50  0000 C CNN
@@
 NoConn ~ 4250 3450
 NoConn ~ 4250 3550
-NoConn ~ 4250 2900
-NoConn ~ 4250 3000
-NoConn ~ 4250 3100
 NoConn ~ 4250 2650
 NoConn ~ 5750 3350
@@
 P 6100 5250
 F 0 "R11" V 6180 5250 50  0000 C CNN
-F 1 "2.2M" V 6100 5250 50  0000 C CNN
+F 1 "100k" V 6100 5250 50  0000 C CNN
 F 2 "Resistors_ThroughHole:Resistor_Horizontal_RM10mm" V 6030 5250 50  0001 C CNN
 F 3 "" H 6100 5250 50  0000 C CNN
@@
 P 6600 4300
 F 0 "R12" V 6680 4300 50  0000 C CNN
-F 1 "2.2M" V 6600 4300 50  0000 C CNN
+F 1 "100k" V 6600 4300 50  0000 C CNN
 F 2 "Resistors_ThroughHole:Resistor_Horizontal_RM10mm" V 6530 4300 50  0001 C CNN
 F 3 "" H 6600 4300 50  0000 C CNN
@@
 	1    0    0    -1
 $EndComp
-NoConn ~ 5750 2550
 $Comp
 L Led_x2 D1
@@
 $Comp
 L VSS #PWR016
-U 1 1 571B05EF
-P 8550 4000
-F 0 "#PWR016" H 8550 3850 50  0001 C CNN
-F 1 "VSS" H 8550 4150 50  0000 C CNN
-F 2 "" H 8550 4000 50  0000 C CNN
-F 3 "" H 8550 4000 50  0000 C CNN
-	1    8550 4000
-	1    0    0    -1
-$EndComp
-$Comp
-L VSS #PWR017
 U 1 1 571B138F
 P 1600 3150
-F 0 "#PWR017" H 1600 3000 50  0001 C CNN
+F 0 "#PWR016" H 1600 3000 50  0001 C CNN
 F 1 "VSS" H 1600 3300 50  0000 C CNN
 F 2 "" H 1600 3150 50  0000 C CNN
@@
 $EndComp
 $Comp
-L VSS #PWR018
+L VSS #PWR017
 U 1 1 571B154F
 P 1900 3950
-F 0 "#PWR018" H 1900 3800 50  0001 C CNN
+F 0 "#PWR017" H 1900 3800 50  0001 C CNN
 F 1 "VSS" H 1900 4100 50  0000 C CNN
 F 2 "" H 1900 3950 50  0000 C CNN
@@
 $EndComp
 $Comp
-L VSS #PWR019
+L VSS #PWR018
 U 1 1 571B18DB
 P 2600 2450
-F 0 "#PWR019" H 2600 2300 50  0001 C CNN
+F 0 "#PWR018" H 2600 2300 50  0001 C CNN
 F 1 "VSS" H 2600 2600 50  0000 C CNN
 F 2 "" H 2600 2450 50  0000 C CNN
@@
 $EndComp
 $Comp
-L VSS #PWR020
+L VSS #PWR019
 U 1 1 571B199A
 P 3700 1950
-F 0 "#PWR020" H 3700 1800 50  0001 C CNN
+F 0 "#PWR019" H 3700 1800 50  0001 C CNN
 F 1 "VSS" H 3700 2100 50  0000 C CNN
 F 2 "" H 3700 1950 50  0000 C CNN
@@
 $EndComp
 $Comp
-L VSS #PWR021
-U 1 1 571B1DEF
-P 6450 3350
-F 0 "#PWR021" H 6450 3200 50  0001 C CNN
-F 1 "VSS" H 6450 3500 50  0000 C CNN
-F 2 "" H 6450 3350 50  0000 C CNN
-F 3 "" H 6450 3350 50  0000 C CNN
-	1    6450 3350
-	1    0    0    -1
-$EndComp
-$Comp
-L GND #PWR022
+L GND #PWR020
 U 1 1 571B25D9
 P 5900 4700
-F 0 "#PWR022" H 5900 4450 50  0001 C CNN
+F 0 "#PWR020" H 5900 4450 50  0001 C CNN
 F 1 "GND" H 5900 4550 50  0000 C CNN
 F 2 "" H 5900 4700 50  0000 C CNN
@@
 $EndComp
 $Comp
-L PWR_FLAG #FLG023
+L PWR_FLAG #FLG021
 U 1 1 571B3284
 P 8350 1750
-F 0 "#FLG023" H 8350 1845 50  0001 C CNN
+F 0 "#FLG021" H 8350 1845 50  0001 C CNN
 F 1 "PWR_FLAG" H 8350 1930 50  0000 C CNN
 F 2 "" H 8350 1750 50  0000 C CNN
@@
 Wire Wire Line
 	8000 1750 8350 1750
-Wire Wire Line
-	6300 3350 6450 3350
 Connection ~ 2100 3950
 Wire Wire Line
@@
 	1450 3150 1600 3150
 Wire Wire Line
-	7100 3900 7300 3900
+	7300 3900 7100 3900
 Connection ~ 8000 1600
 Wire Wire Line
@@
 Wire Wire Line
 	3350 3650 3350 3350
-Connection ~ 9000 3500
-Wire Wire Line
-	9050 3500 9000 3500
 Connection ~ 6600 4600
 Wire Wire Line
@@
 Wire Wire Line
 	5150 4600 5150 4500
-Connection ~ 8850 4000
 Wire Wire Line
 	9000 4000 9000 3400
@@
 	9000 3400 9050 3400
 Wire Wire Line
-	8550 4000 9000 4000
-Wire Wire Line
-	8850 3950 8850 4000
+	8850 4000 9000 4000
+Wire Wire Line
+	8850 3950 8850 4200
 Wire Wire Line
 	8850 3300 8850 3650
@@
 	1450 2900 1450 3150
 Wire Wire Line
-	1300 2700 1550 2700
+	1300 2700 1600 2700
 Wire Wire Line
 	1450 2700 1450 2550
@@
 Connection ~ 1450 2700
 Wire Wire Line
-	1850 2700 1950 2700
+	1800 2700 1950 2700
 Wire Wire Line
 	2250 2700 2400 2700
@@
 Connection ~ 3150 2800
 Wire Wire Line
-	5750 2800 6300 2800
-Wire Wire Line
-	6300 2800 6300 2950
-Wire Wire Line
-	6300 3250 6300 3350
-Wire Wire Line
-	6450 3100 6550 3100
+	5750 2800 6350 2800
+Wire Wire Line
+	6350 2800 6350 2950
+Wire Wire Line
+	6350 3250 6350 3600
+Wire Wire Line
+	6500 3100 6550 3100
 Wire Wire Line
 	6850 3100 6950 3100
@@
 Connection ~ 7300 3100
 Wire Wire Line
-	7300 3900 7300 3500
+	7300 3500 7300 3900
 Wire Wire Line
 	4250 3250 3050 3250
@@
 Text Label 8900 3300 0    60   ~ 0
 VREF
+Connection ~ 8850 4000
+$Comp
+L GND #PWR022
+U 1 1 572CAC9C
+P 8850 4200
+F 0 "#PWR022" H 8850 3950 50  0001 C CNN
+F 1 "GND" H 8850 4050 50  0000 C CNN
+F 2 "" H 8850 4200 50  0000 C CNN
+F 3 "" H 8850 4200 50  0000 C CNN
+	1    8850 4200
+	1    0    0    -1
+$EndComp
+Wire Wire Line
+	6350 3600 7300 3600
+Connection ~ 7300 3600
+Wire Wire Line
+	5750 2550 5950 2550
+Wire Wire Line
+	5950 2550 5950 2900
+Wire Wire Line
+	5950 2900 6200 2900
+Wire Wire Line
+	6200 2900 6200 3700
+Wire Wire Line
+	6200 3700 6950 3700
+Wire Wire Line
+	6950 3700 6950 4100
+Wire Wire Line
+	6950 4100 8500 4100
+Wire Wire Line
+	8500 4100 8500 3500
+Wire Wire Line
+	8500 3500 9050 3500
+Text Label 7650 4100 0    60   ~ 0
+DO3
+$Comp
+L VCC #PWR023
+U 1 1 572D38F0
+P 3700 2700
+F 0 "#PWR023" H 3700 2550 50  0001 C CNN
+F 1 "VCC" H 3700 2850 50  0000 C CNN
+F 2 "" H 3700 2700 50  0000 C CNN
+F 3 "" H 3700 2700 50  0000 C CNN
+	1    3700 2700
+	1    0    0    -1
+$EndComp
+Wire Wire Line
+	3700 2700 3700 3100
+Wire Wire Line
+	3700 2900 4250 2900
+Wire Wire Line
+	3700 3000 4250 3000
+Connection ~ 3700 2900
+Wire Wire Line
+	3700 3100 4250 3100
+Connection ~ 3700 3000
 $EndSCHEMATC

Commit message: Swapped DO3 and DO4. Assign CE# to DO4.
Parts:
- R9: value 100 -> 22k; footprint Resistors_ThroughHole:Resistor_Horizontal_RM10mm -> Resistors_SMD:R_0603_HandSoldering
Connections:
- net labels added: DO4
- net labels removed: DO3
- wire segments 129 -> 128
Changed lines of the file:
@@
 P 8350 3200
 F 0 "R9" V 8430 3200 50  0000 C CNN
-F 1 "100" V 8350 3200 50  0000 C CNN
-F 2 "Resistors_ThroughHole:Resistor_Horizontal_RM10mm" V 8280 3200 50  0001 C CNN
+F 1 "22k" V 8350 3200 50  0000 C CNN
+F 2 "Resistors_SMD:R_0603_HandSoldering" V 8280 3200 50  0001 C CNN
 F 3 "" H 8350 3200 50  0000 C CNN
 	1    8350 3200
@@
 P 6250 2350
 F 0 "D1" H 6250 2575 50  0000 C CNN
-F 1 "Led_x2" H 6250 2100 50  0000 C CNN
+F 1 "Led_x2" H 6000 2550 50  0000 C CNN
 F 2 "favorites:LED-3MM" H 6250 2350 50  0001 C CNN
 F 3 "" H 6250 2350 50  0000 C CNN
@@
 	6100 4900 6100 5100
 Wire Wire Line
-	6100 2650 6100 4600
-Wire Wire Line
-	5750 2650 6100 2650
+	6100 2550 6100 4600
 Wire Wire Line
 	4950 4200 4950 4600
@@
 	3300 1950 3350 1950
 Wire Wire Line
-	3150 2100 3150 2800
-Wire Wire Line
-	3000 2800 4250 2800
+	3150 2100 3150 3000
 Wire Wire Line
 	3650 1950 3700 1950
@@
 Connection ~ 7300 3600
 Wire Wire Line
-	5750 2550 5950 2550
-Wire Wire Line
-	5950 2550 5950 2900
-Wire Wire Line
-	5950 2900 6200 2900
-Wire Wire Line
-	6200 2900 6200 3700
+	5750 2550 6100 2550
+Wire Wire Line
+	6200 2650 6200 3700
 Wire Wire Line
 	6200 3700 6950 3700
@@
 	8500 3500 9050 3500
 Text Label 7650 4100 0    60   ~ 0
-DO3
+DO4
 $Comp
 L VCC #PWR023
@@
 	3700 2900 4250 2900
 Wire Wire Line
-	3700 3000 4250 3000
+	3150 2800 3000 2800
 Connection ~ 3700 2900
 Wire Wire Line
 	3700 3100 4250 3100
-Connection ~ 3700 3000
+Wire Wire Line
+	3150 3000 4250 3000
+Wire Wire Line
+	4250 2800 3700 2800
+Connection ~ 3700 2800
+Wire Wire Line
+	5750 2650 6200 2650
 $EndSCHEMATC
