File: KiCad/AppAudio.sch (KiCad schematic (older format))
At the start: 33 parts, among them P1 WRITER-VCC, Q1 Q_NMOS_SGD, SW1 SW_PUSH, SW2 SW_PUSH, U1 TWE_LITE_SMD, U2 NJM13404, U3 HT82V739

Commit message: Replaced some SMD registers.
Parts:
- added R14, R15, R4: 510, Resistors_SMD:R_0603_HandSoldering, symbol R
- R10, R13: value 1k -> 510
- R11: value 100k -> 1M
- R16: renamed from R3; value 1.5k -> 510
- R3: renamed from R4; value 1k -> 510
Connections:
- wire segments 128 -> 136
Other:
- moved on the sheet: U2A, U2B

Commit message: Assign LED1 as TX indicator.
Parts:
- added R17: 510, Resistors_SMD:R_0603_HandSoldering, symbol R
Connections:
- net labels added: CE#
- net labels removed: DO4
- wire segments 136 -> 137

Commit message: Use MEMS mic and passive LPF.
Parts:
- removed C1: 22u, Capacitors_ThroughHole:C_Radial_D6.3_L11.2_P2.5, symbol C_Small
- removed C2: 0.1u, Capacitors_ThroughHole:C_Rect_L4_W2.5_P2.5, symbol C_Small
- removed C4: 3300p, Capacitors_ThroughHole:C_Rect_L4_W2.5_P2.5, symbol C_Small
- removed C5: 1000p, Capacitors_ThroughHole:C_Rect_L4_W2.5_P2.5, symbol C_Small
- removed MIC1: MIC_ELECTRET, favorites:DB-C9767, symbol MIC_ELECTRET
- removed Q1: Q_NMOS_SGD, favorites:EMT3, symbol Q_NMOS_SGD
- removed R1, R2: 10k, Resistors_SMD:R_0603_HandSoldering, symbol R
- removed R10, R14, R15, R16, R17, R3, R4: 510, Resistors_SMD:R_0603_HandSoldering, symbol R
- removed R11: 1M, Resistors_ThroughHole:Resistor_Horizontal_RM10mm, symbol R
- removed R12: 100k, Resistors_ThroughHole:Resistor_Horizontal_RM10mm, symbol R
- removed R8, R9: 22k, Resistors_SMD:R_0603_HandSoldering, symbol R
- removed U2: NJM13404, Housings_DIP:DIP-8_W7.62mm, symbol LMC6062
- removed VR1: 50k, favorites:RV-3362P, symbol POT
- removed VR2: 1k, favorites:RV-3362P, symbol POT
- added C1: 0.047u, Capacitors_ThroughHole:C_Rect_L4_W2.5_P2.5, symbol C
- added C2: 0.01u, Capacitors_ThroughHole:C_Rect_L4_W2.5_P2.5, symbol C
- added RV1: 1k, symbol POT
- added U1: AE-SPU0414, symbol AE-SPU0414
- C3: value 220u -> 47u
- C4: renamed from C6; value 22u -> 1u
- R5: value 57k -> 1k; footprint Resistors_SMD:R_0603_HandSoldering -> Resistors_ThroughHole:Resistor_Horizontal_RM10mm
- R6: value 10k -> 4.7k; footprint Resistors_SMD:R_0603_HandSoldering -> Resistors_ThroughHole:Resistor_Horizontal_RM10mm
- R7: value 22k -> 10k; footprint Resistors_SMD:R_0603_HandSoldering -> Resistors_ThroughHole:Resistor_Horizontal_RM10mm
- renumbered C7 to C5, R13 to R4, U1 to U2
Connections:
- net labels added: MIC_VDD
- net labels removed: QGND, VSS
- wire segments 137 -> 88
- no-connect marks 14 -> 15
